File: pickit2_adapter.kicad_pcb (KiCad board)
At the start: 2 copper layers, 35.8 x 35.8 mm, 7 parts

Commit message: Fixed mask
Other:
- board text added: "ICSP"
- board text added: "PICkit2 to AVR ICSP/SPI FLASH adapter"
- board text removed: "ISCP"
- board text removed: "PICkit2 to AVR ISCP/SPI FLASH adapter"
Changed lines of the file:
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@@
     )
   )
-  (gr_text ISCP (at 100.838 66.421) (layer F.SilkS)
+  (gr_text ICSP (at 100.838 66.421) (layer F.SilkS)
     (effects (font (size 1 1) (thickness 0.15)))
   )
@@
     (effects (font (size 0.6 0.6) (thickness 0.13)))
   )
-  (gr_text "PICkit2 to AVR ISCP/SPI FLASH adapter" (at 91.059 69.596) (layer F.SilkS)
+  (gr_text "PICkit2 to AVR ICSP/SPI FLASH adapter" (at 91.059 69.596) (layer F.SilkS)
     (effects (font (size 0.6 0.6) (thickness 0.13)))
   )
